File: kicad/pcbs/main_pcb.kicad_pcb (KiCad board)
At the start: 2 copper layers, 267 x 98.4 mm, 82 parts

Commit message: Adjust PCB component positions
Parts:
- added G*** (x2): LOGO, LOGO, B.Cu at (0.00, 0.00)
- added H1: , ceoloide:mounting_hole_plated, F.Cu at (56.0, 55.0)
- added H2: , ceoloide:mounting_hole_plated, F.Cu at (128.5, 46.4)
- added H3: , ceoloide:mounting_hole_plated, F.Cu at (84.0, 94.7)
- added H4: , ceoloide:mounting_hole_plated, F.Cu at (136.5, 104.1)
- added H5: , ceoloide:mounting_hole_plated, F.Cu at (286.0, 55.0)
- added H6: , ceoloide:mounting_hole_plated, F.Cu at (213.5, 46.4)
- added H7: , ceoloide:mounting_hole_plated, F.Cu at (258.0, 94.7)
- added H8: , ceoloide:mounting_hole_plated, F.Cu at (205.5, 104.1)
- D1, D10, D11, D12, D13, D14, D15, D16, D17, D18, D19, D2, D20, D21, D22, D23, D24, D25, D26, D27, D28, D29, D3, D30, D31, D32, D33, D34, D35, D36, D4, D5, D6, D7, D8, D9: moved to F.Cu
- moved PWR1 6.00 mm to (150.5, 45.4)
- moved PWR2 6.00 mm to (191.5, 45.4)
- moved JST1 4.47 mm to (144.5, 102.1)
- moved JST2 4.47 mm to (197.5, 102.1)
- moved DISP1 2.00 mm to (146.5, 76.1)
- moved DISP2 2.00 mm to (195.5, 76.1)
Other:
- outline, holes or cut-outs redrawn
- board text added: "n1tsu"

Commit message: Update README
Parts:
- removed G*** (x2): LOGO, LOGO

Commit message: Remove pcb border
Parts:
- removed H7, H8: , ceoloide:mounting_hole_plated
- moved H5 104.4 mm to (181.7, 50.4)
- moved H4 92.6 mm to (211.9, 50.4)
- moved H1 74.2 mm to (130.1, 50.4)
- moved H6 58.3 mm to (205.1, 104.1)
- moved H3 53.7 mm to (136.9, 104.1)
- moved H2 32.1 mm to (160.3, 50.4)
- moved D36 4.67 mm to (205.9, 114.1)
- moved RST1 4.47 mm to (138.5, 49.4)
- moved RST2 4.47 mm to (203.5, 49.4)
- moved D18 4.09 mm to (136.6, 114.3)
- moved S18 4.09 mm to (135.5, 116.5)
- moved S36 4.09 mm to (206.5, 116.5)
- moved DISP1 4.00 mm to (146.5, 80.1)
- moved DISP2 4.00 mm to (195.5, 80.1)
- moved MCU1 4.00 mm to (146.5, 62.3)
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Other:
- board size 267 x 98.4 mm -> 259 x 86.8 mm
- board text added: "n36tsu v0.1.0"
- board text removed: "n1tsu"

Commit message: Route left PCB
Connections:
- net CS renamed P02
- DISP1 pad 4: SCK -> P029
- DISP1 pad 5: MOSI -> P031
- DISP2 pad 4: SCK -> P029
- DISP2 pad 5: MOSI -> P031
- S1 pad 1: matrix_qcolumn_zrow -> qcolumn_zrow
- S1 pad 2: GND -> (no net)
- S10 pad 1: matrix_rcolumn_zrow -> rcolumn_zrow
- S10 pad 2: GND -> (no net)
- S11 pad 1: matrix_rcolumn_arow -> rcolumn_arow
- S11 pad 2: GND -> (no net)
- S12 pad 1: matrix_rcolumn_qrow -> rcolumn_qrow
- S12 pad 2: GND -> (no net)
- S13 pad 1: matrix_tcolumn_zrow -> tcolumn_zrow
- S13 pad 2: GND -> (no net)
- S14 pad 1: matrix_tcolumn_arow -> tcolumn_arow
- S14 pad 2: GND -> (no net)
- S15 pad 1: matrix_tcolumn_qrow -> tcolumn_qrow
- S15 pad 2: GND -> (no net)
- S16 pad 1: thumb_inner -> inner_default
- S16 pad 2: GND -> (no net)
- S17 pad 1: thumb_middle -> middle_default
- S17 pad 2: GND -> (no net)
- S18 pad 1: thumb_outer -> outer_default
- S18 pad 2: GND -> (no net)
- S19 pad 1: mirror_matrix_qcolumn_zrow -> mirror_qcolumn_zrow
- S19 pad 2: GND -> (no net)
- S2 pad 1: matrix_qcolumn_arow -> qcolumn_arow
- S2 pad 2: GND -> (no net)
- S20 pad 1: mirror_matrix_qcolumn_arow -> mirror_qcolumn_arow
- S20 pad 2: GND -> (no net)
- S21 pad 1: mirror_matrix_qcolumn_qrow -> mirror_qcolumn_qrow
- S21 pad 2: GND -> (no net)
- S22 pad 1: mirror_matrix_wcolumn_zrow -> mirror_wcolumn_zrow
- S22 pad 2: GND -> (no net)
- S23 pad 1: mirror_matrix_wcolumn_arow -> mirror_wcolumn_arow
- S23 pad 2: GND -> (no net)
- S24 pad 1: mirror_matrix_wcolumn_qrow -> mirror_wcolumn_qrow
- S24 pad 2: GND -> (no net)
- S25 pad 1: mirror_matrix_ecolumn_zrow -> mirror_ecolumn_zrow
- S25 pad 2: GND -> (no net)
- S26 pad 1: mirror_matrix_ecolumn_arow -> mirror_ecolumn_arow
- S26 pad 2: GND -> (no net)
- S27 pad 1: mirror_matrix_ecolumn_qrow -> mirror_ecolumn_qrow
- S27 pad 2: GND -> (no net)
- S28 pad 1: mirror_matrix_rcolumn_zrow -> mirror_rcolumn_zrow
- S28 pad 2: GND -> (no net)
- S29 pad 1: mirror_matrix_rcolumn_arow -> mirror_rcolumn_arow
- S29 pad 2: GND -> (no net)
- S3 pad 1: matrix_qcolumn_qrow -> qcolumn_qrow
- S3 pad 2: GND -> (no net)
- S30 pad 1: mirror_matrix_rcolumn_qrow -> mirror_rcolumn_qrow
- S30 pad 2: GND -> (no net)
- S31 pad 1: mirror_matrix_tcolumn_zrow -> mirror_tcolumn_zrow
- S31 pad 2: GND -> (no net)
- S32 pad 1: mirror_matrix_tcolumn_arow -> mirror_tcolumn_arow
- S32 pad 2: GND -> (no net)
- S33 pad 1: mirror_matrix_tcolumn_qrow -> mirror_tcolumn_qrow
- S33 pad 2: GND -> (no net)
- S34 pad 1: mirror_thumb_inner -> mirror_inner_default
- S34 pad 2: GND -> (no net)
- S35 pad 1: mirror_thumb_middle -> mirror_middle_default
- S35 pad 2: GND -> (no net)
- S36 pad 1: mirror_thumb_outer -> mirror_outer_default
- S36 pad 2: GND -> (no net)
- S4 pad 1: matrix_wcolumn_zrow -> wcolumn_zrow
- S4 pad 2: GND -> (no net)
- S5 pad 1: matrix_wcolumn_arow -> wcolumn_arow
- S5 pad 2: GND -> (no net)
- S6 pad 1: matrix_wcolumn_qrow -> wcolumn_qrow
- S6 pad 2: GND -> (no net)
- S7 pad 1: matrix_ecolumn_zrow -> ecolumn_zrow
- S7 pad 2: GND -> (no net)
- S8 pad 1: matrix_ecolumn_arow -> ecolumn_arow
- S8 pad 2: GND -> (no net)
- S9 pad 1: matrix_ecolumn_qrow -> ecolumn_qrow
- S9 pad 2: GND -> (no net)

Commit message: Modify routing
Parts:
- moved H1 0.30 mm to (130.1, 50.7)
- moved H2 0.30 mm to (160.3, 50.7)
- moved H4 0.30 mm to (211.9, 50.7)
- moved H5 0.30 mm to (181.7, 50.7)
- moved PWR1 0.30 mm to (150.5, 49.7)
- moved PWR2 0.30 mm to (191.5, 49.7)
- moved RST1 0.30 mm to (138.5, 49.7)
- moved RST2 0.30 mm to (203.5, 49.7)
Connections:
- DISP1 pad 1: P02 -> P017
- DISP1 pad 2: GND -> P020
- DISP1 pad 4: P029 -> GND
- DISP1 pad 5: P031 -> P022
- DISP2 pad 1: P02 -> P017
- DISP2 pad 2: GND -> P020
- DISP2 pad 4: P029 -> GND
- DISP2 pad 5: P031 -> P022
Changed lines of the file:
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@@
   (title_block
     (title "main_pcb")
-    (date "2024-12-14")
+    (date "2024-12-16")
     (rev "0.0.1")
     (company "n1tsu")
@@
 (net 65 "JST2_1")
 (net 66 "JST2_2")
-(net 67 "P02")
-(net 68 "DISP1_1")
-(net 69 "DISP1_2")
-(net 70 "DISP1_4")
-(net 71 "DISP1_5")
-(net 72 "DISP2_1")
-(net 73 "DISP2_2")
-(net 74 "DISP2_4")
-(net 75 "DISP2_5")
+(net 67 "DISP1_1")
+(net 68 "DISP1_2")
+(net 69 "DISP1_4")
+(net 70 "DISP1_5")
+(net 71 "DISP2_1")
+(net 72 "DISP2_2")
+(net 73 "DISP2_4")
+(net 74 "DISP2_5")
 (footprint "CPG1316S01D02_mikeholscher"
   (layer "F.Cu")
@@
   (footprint "ceoloide:power_switch_smd_side"
     (layer "F.Cu")
-    (at 150.5 49.394499999999994 90)
+    (at 150.5 49.69449999999999 90)
     (property "Reference" "PWR1"
       (at -3.6 0 0)
@@
   (footprint "ceoloide:power_switch_smd_side"
     (layer "F.Cu")
-    (at 191.5 49.394499999999994 90)
+    (at 191.5 49.69449999999999 90)
     (property "Reference" "PWR2"
       (at -3.6 0 0)
@@
   (footprint "ceoloide:reset_switch_smd_side"
     (layer "F.Cu")
-    (at 138.5 49.394499999999994 0)
+    (at 138.5 49.69449999999999 0)
     (property "Reference" "RST1"
       (at 0 0 0)
@@
     (fp_line (start 1.3 -2.75) (end 1.3 -1.75) (stroke (width 0.1) (type solid)) (layer "Dwgs.User"))
     (fp_line (start 2.35 -1.75) (end 2.35 1.75) (stroke (width 0.1) (type solid)) (layer "Dwgs.User"))
+    (pad "" np_thru_hole circle (at 0 -1.375 180) (size 0.75 0.75) (drill 0.75) (layers "*.Cu" "*.Mask"))
+    (pad "" np_thru_hole circle (at 0 1.375 180) (size 0.75 0.75) (drill 0.75) (layers "*.Cu" "*.Mask"))
     (pad "1" smd rect (at 2.625 -0.85 180) (size 1.55 1) (layers "F.Cu" "F.Paste" "F.Mask") (net 38 "GND"))
     (pad "2" smd rect (at 2.625 0.85 180) (size 1.55 1) (layers "F.Cu" "F.Paste" "F.Mask") (net 39 "RST"))
@@
   (footprint "ceoloide:reset_switch_smd_side"
     (layer "F.Cu")
-    (at 203.5 49.394499999999994 0)
+    (at 203.5 49.69449999999999 0)
     (property "Reference" "RST2"
       (at 0 0 0)
@@
     (fp_line (start 1.3 -2.75) (end 1.3 -1.75) (stroke (width 0.1) (type solid)) (layer "Dwgs.User"))
     (fp_line (start 2.35 -1.75) (end 2.35 1.75) (stroke (width 0.1) (type solid)) (layer "Dwgs.User"))
+    (pad "" np_thru_hole circle (at 0 -1.375 180) (size 0.75 0.75) (drill 0.75) (layers "*.Cu" "*.Mask"))
+    (pad "" np_thru_hole circle (at 0 1.375 180) (size 0.75 0.75) (drill 0.75) (layers "*.Cu" "*.Mask"))
     (pad "1" smd rect (at 2.625 -0.85 180) (size 1.55 1) (layers "F.Cu" "F.Paste" "F.Mask") (net 38 "GND"))
     (pad "2" smd rect (at 2.625 0.85 180) (size 1.55 1) (layers "F.Cu" "F.Paste" "F.Mask") (net 39 "RST"))
@@
     (fp_line (start 6.41 15.37) (end 6.41 18.03) (layer "F.SilkS") (stroke (width 0.12) (type solid)))
     (fp_line (start 6.41 15.37) (end -6.41 15.37) (layer "F.SilkS") (stroke (width 0.12) (type solid)))
-    (fp_text user "DA" (at -5.08 13.1 -90) (layer "F.SilkS")
-      (effects (font (size 1 1) (thickness 0.15)))
-    )
-    (fp_text user "CS" (at 5.12 13.1 -90) (layer "F.SilkS")
-      (effects (font (size 1 1) (thickness 0.15)))
-    )
-    (fp_text user "GND" (at 2.62 13.1 -90) (layer "F.SilkS")
-      (effects (font (size 1 1) (thickness 0.15)))
-    )
-    (fp_text user "VCC" (at 0.15 14.6 -90) (layer "F.SilkS")
-      (effects (font (size 1 1) (thickness 0.15)))
-    )
-    (fp_text user "CL" (at -2.48 13.1 -90) (layer "F.SilkS")
-      (effects (font (size 1 1) (thickness 0.15)))
+    (fp_text user "P017" (at -5.08 18.5 0) (unlocked yes) (layer "F.SilkS")
+      (effects (font (size 1 1) (thickness 0.15)) (justify right))
+    )
+    (fp_text user "P020" (at -2.48 18.5 0) (unlocked yes) (layer "F.SilkS")
+      (effects (font (size 1 1) (thickness 0.15)) (justify right))
+    )
+    (fp_text user "VCC" (at 0.15 18.5 0) (unlocked yes) (layer "F.SilkS")
+      (effects (font (size 1 1) (thickness 0.15)) (justify right))
+    )
+    (fp_text user "GND" (at 2.62 18.5 0) (unlocked yes) (layer "F.SilkS")
+      (effects (font (size 1 1) (thickness 0.15)) (justify right))
+    )
+    (fp_text user "P022" (at 5.12 18.5 0) (unlocked yes) (layer "F.SilkS")
+      (effects (font (size 1 1) (thickness 0.15)) (justify right))
     )
     (fp_line (start 6.88 14.9) (end 6.88 18.45) (layer "F.CrtYd") (stroke (width 0.15) (type solid)))
@@
     (fp_line (start -6.82 18.45) (end -6.82 14.9) (layer "F.CrtYd") (stroke (width 0.15) (type solid)))
     (fp_line (start -6.82 14.9) (end 6.88 14.9) (layer "F.CrtYd") (stroke (width 0.15) (type solid)))
-    (pad "1" smd oval (at -5.08 16.7 180) (size 1.7 1.7) (drill 1) (layers "F.Cu" "F.Mask") (net 67 "P02"))
-    (pad "2" smd oval (at -2.54 16.7 180) (size 1.7 1.7) (drill 1) (layers "F.Cu" "F.Mask") (net 38 "GND"))
-    (pad "3" smd oval (at 0 16.7 180) (size 1.7 1.7) (drill 1) (layers "F.Cu" "F.Mask") (net 40 "VCC"))
-    (pad "4" smd oval (at 2.54 16.7 180) (size 1.7 1.7) (drill 1) (layers "F.Cu" "F.Mask") (net 42 "P029"))
-    (pad "5" smd circle (at 5.08 16.7 180) (size 1.7 1.7) (drill 1) (layers "F.Cu" "F.Mask") (net 41 "P031"))
+    (pad "1" thru_hole oval (at -5.08 16.7 180) (size 1.7 1.7) (drill 1) (layers "*.Cu" "*.Mask") (net 51 "P017"))
+    (pad "2" thru_hole oval (at -2.54 16.7 180) (size 1.7 1.7) (drill 1) (layers "*.Cu" "*.Mask") (net 52 "P020"))
+    (pad "3" thru_hole oval (at 0 16.7 180) (size 1.7 1.7) (drill 1) (layers "*.Cu" "*.Mask") (net 40 "VCC"))
+    (pad "4" thru_hole oval (at 2.54 16.7 180) (size 1.7 1.7) (drill 1) (layers "*.Cu" "*.Mask") (net 38 "GND"))
+    (pad "5" thru_hole circle (at 5.08 16.7 180) (size 1.7 1.7) (drill 1) (layers "*.Cu" "*.Mask") (net 53 "P022"))
     (fp_line (start 5.4 13.4) (end 5.4 -11.9) (layer Dwgs.User) (stroke (width 0.15) (type solid)))
     (fp_line (start -5.4 13.4) (end -5.4 -11.9) (layer Dwgs.User) (stroke (width 0.15) (type solid)))
@@
     (fp_line (start 6.41 15.37) (end 6.41 18.03) (layer "F.SilkS") (stroke (width 0.12) (type solid)))
     (fp_line (start 6.41 15.37) (end -6.41 15.37) (layer "F.SilkS") (stroke (width 0.12) (type solid)))
-    (fp_text user "DA" (at -5.08 13.1 90) (layer "F.SilkS")
-      (effects (font (size 1 1) (thickness 0.15)))
-    )
-    (fp_text user "CS" (at 5.12 13.1 90) (layer "F.SilkS")
-      (effects (font (size 1 1) (thickness 0.15)))
-    )
-    (fp_text user "GND" (at 2.62 13.1 90) (layer "F.SilkS")
-      (effects (font (size 1 1) (thickness 0.15)))
-    )
-    (fp_text user "VCC" (at 0.15 14.6 90) (layer "F.SilkS")
-      (effects (font (size 1 1) (thickness 0.15)))
-    )
-    (fp_text user "CL" (at -2.48 13.1 90) (layer "F.SilkS")
-      (effects (font (size 1 1) (thickness 0.15)))
+    (fp_text user "P017" (at -5.08 18.5 180) (unlocked yes) (layer "F.SilkS")
+      (effects (font (size 1 1) (thickness 0.15)) (justify right))
+    )
+    (fp_text user "P020" (at -2.48 18.5 180) (unlocked yes) (layer "F.SilkS")
+      (effects (font (size 1 1) (thickness 0.15)) (justify right))
+    )
+    (fp_text user "VCC" (at 0.15 18.5 180) (unlocked yes) (layer "F.SilkS")
+      (effects (font (size 1 1) (thickness 0.15)) (justify right))
+    )
+    (fp_text user "GND" (at 2.62 18.5 180) (unlocked yes) (layer "F.SilkS")
+      (effects (font (size 1 1) (thickness 0.15)) (justify right))
+    )
+    (fp_text user "P022" (at 5.12 18.5 180) (unlocked yes) (layer "F.SilkS")
+      (effects (font (size 1 1) (thickness 0.15)) (justify right))
     )
     (fp_line (start 6.88 14.9) (end 6.88 18.45) (layer "F.CrtYd") (stroke (width 0.15) (type solid)))
@@
     (fp_line (start -6.82 18.45) (end -6.82 14.9) (layer "F.CrtYd") (stroke (width 0.15) (type solid)))
     (fp_line (start -6.82 14.9) (end 6.88 14.9) (layer "F.CrtYd") (stroke (width 0.15) (type solid)))
-    (pad "1" smd oval (at -5.08 16.7 360) (size 1.7 1.7) (drill 1) (layers "F.Cu" "F.Mask") (net 67 "P02"))
-    (pad "2" smd oval (at -2.54 16.7 360) (size 1.7 1.7) (drill 1) (layers "F.Cu" "F.Mask") (net 38 "GND"))
-    (pad "3" smd oval (at 0 16.7 360) (size 1.7 1.7) (drill 1) (layers "F.Cu" "F.Mask") (net 40 "VCC"))
-    (pad "4" smd oval (at 2.54 16.7 360) (size 1.7 1.7) (drill 1) (layers "F.Cu" "F.Mask") (net 42 "P029"))
-    (pad "5" smd circle (at 5.08 16.7 360) (size 1.7 1.7) (drill 1) (layers "F.Cu" "F.Mask") (net 41 "P031"))
+    (pad "1" thru_hole oval (at -5.08 16.7 360) (size 1.7 1.7) (drill 1) (layers "*.Cu" "*.Mask") (net 51 "P017"))
+    (pad "2" thru_hole oval (at -2.54 16.7 360) (size 1.7 1.7) (drill 1) (layers "*.Cu" "*.Mask") (net 52 "P020"))
+    (pad "3" thru_hole oval (at 0 16.7 360) (size 1.7 1.7) (drill 1) (layers "*.Cu" "*.Mask") (net 40 "VCC"))
+    (pad "4" thru_hole oval (at 2.54 16.7 360) (size 1.7 1.7) (drill 1) (layers "*.Cu" "*.Mask") (net 38 "GND"))
+    (pad "5" thru_hole circle (at 5.08 16.7 360) (size 1.7 1.7) (drill 1) (layers "*.Cu" "*.Mask") (net 53 "P022"))
     (fp_line (start 5.4 13.4) (end 5.4 -11.9) (layer Dwgs.User) (stroke (width 0.15) (type solid)))
     (fp_line (start -5.4 13.4) (end -5.4 -11.9) (layer Dwgs.User) (stroke (width 0.15) (type solid)))
@@
   (footprint "ceoloide:mounting_hole_plated"
     (layer "F.Cu")
-    (at 130.1 50.394499999999994 0)
+    (at 130.1 50.69449999999999 0)
     (property "Reference" "H1"
       (at 0 3 0)
@@
   (footprint "ceoloide:mounting_hole_plated"
     (layer "F.Cu")
-    (at 160.3 50.394499999999994 0)
+    (at 160.3 50.69449999999999 0)
     (property "Reference" "H2"
       (at 0 3 0)
@@
   (footprint "ceoloide:mounting_hole_plated"
     (layer "F.Cu")
-    (at 211.9 50.394499999999994 0)
+    (at 211.9 50.69449999999999 0)
     (property "Reference" "H4"
       (at 0 3 0)
@@
   (footprint "ceoloide:mounting_hole_plated"
     (layer "F.Cu")
-    (at 181.7 50.394499999999994 0)
+    (at 181.7 50.69449999999999 0)
     (property "Reference" "H5"
       (at 0 3 0)
