File: kicad/pcbs/main_pcb_routed.kicad_pcb (KiCad board)
At the start: 2 copper layers, 259 x 86.8 mm, 88 parts

Commit message: Complete PCB wiring
Parts:
- moved H1 0.30 mm to (130.1, 50.7)
- moved H2 0.30 mm to (160.3, 50.7)
- moved H4 0.30 mm to (211.9, 50.7)
- moved H5 0.30 mm to (181.7, 50.7)
- moved PWR1 0.30 mm to (150.5, 49.7)
- moved PWR2 0.30 mm to (191.5, 49.7)
- moved RST1 0.30 mm to (138.5, 49.7)
- moved RST2 0.30 mm to (203.5, 49.7)
Connections:
- D1 pad 1: (no net) -> P011
- D10 pad 1: (no net) -> P011
- D11 pad 1: (no net) -> P104
- D13 pad 1: (no net) -> P011
- D14 pad 1: (no net) -> P104
- D16 pad 1: (no net) -> P100
- D17 pad 1: (no net) -> P100
- D18 pad 1: (no net) -> P100
- D19 pad 1: (no net) -> P011
- D2 pad 1: (no net) -> P104
- D20 pad 1: (no net) -> P104
- D21 pad 1: (no net) -> P106
- D22 pad 1: (no net) -> P011
- D23 pad 1: (no net) -> P104
- D24 pad 1: (no net) -> P106
- D25 pad 1: (no net) -> P011
- D26 pad 1: (no net) -> P104
- D27 pad 1: (no net) -> P106
- D28 pad 1: (no net) -> P011
- D29 pad 1: (no net) -> P104
- D30 pad 1: (no net) -> P106
- D31 pad 1: (no net) -> P011
- D32 pad 1: (no net) -> P104
- D33 pad 1: (no net) -> P106
- D34 pad 1: (no net) -> P100
- D35 pad 1: (no net) -> P100
- D36 pad 1: (no net) -> P100
- D4 pad 1: (no net) -> P011
- D5 pad 1: (no net) -> P104
- D7 pad 1: (no net) -> P011
- D8 pad 1: (no net) -> P104
- DISP1 pad 1: P002 -> P017
- DISP1 pad 2: GND -> P020
- DISP1 pad 4: P029 -> GND
- DISP1 pad 5: P031 -> P022
- DISP2 pad 1: P02 -> P017
- DISP2 pad 2: GND -> P020
- DISP2 pad 4: P029 -> GND
- DISP2 pad 5: P031 -> P022
- S1 pad 2: P022 -> P115
- S10 pad 2: (no net) -> P010
- S11 pad 2: (no net) -> P010
- S12 pad 2: (no net) -> P010
- S13 pad 2: P006 -> P009
- S14 pad 2: P006 -> P009
- S15 pad 2: P006 -> P009
- S16 pad 2: P017 -> P111
- S17 pad 2: (no net) -> P010
- S18 pad 2: P006 -> P009
- S19 pad 2: (no net) -> P115
- S2 pad 2: P022 -> P115
- S20 pad 2: (no net) -> P115
- S21 pad 2: (no net) -> P115
- S22 pad 2: (no net) -> P113
- S23 pad 2: (no net) -> P113
- S24 pad 2: (no net) -> P113
- S25 pad 2: (no net) -> P111
- S26 pad 2: (no net) -> P111
- S27 pad 2: (no net) -> P111
- S28 pad 2: (no net) -> P010
- S29 pad 2: (no net) -> P010
- S3 pad 2: P022 -> P115
- S30 pad 2: (no net) -> P010
- S31 pad 2: (no net) -> P009
- S32 pad 2: (no net) -> P009
- S33 pad 2: (no net) -> P009
- S34 pad 2: (no net) -> P111
- S35 pad 2: (no net) -> P010
- S36 pad 2: (no net) -> P009
- S4 pad 2: P020 -> P113
- S5 pad 2: P020 -> P113
- S5 pad 3: P022 -> (no net)
- S6 pad 2: P020 -> P113
- S7 pad 2: P017 -> P111
- S8 pad 2: P017 -> P111
- S9 pad 2: P017 -> P111
Routing:
- net P011: track 0.00 -> 276.2 mm, vias 0 -> 12
- net P115: track 0.00 -> 268.6 mm, vias 0 -> 4
- net P104: track 0.00 -> 235.6 mm, vias 0 -> 12
- net P100: track 0.00 -> 225.2 mm, vias 0 -> 8
- net P113: track 0.00 -> 222.7 mm, vias 0 -> 4
- net P111: track 98.1 -> 251.3 mm
- net (no net): track 127.2 -> 0.52 mm, vias 2 -> 0
- net P006: track 122.5 -> 0.00 mm
- net P106: track 119.5 -> 233.2 mm, vias 6 -> 12
- net GND: track 121.0 -> 230.7 mm, vias 2 -> 0
- net P010: track 122.9 -> 212.8 mm, vias 2 -> 4
- net BAT_P: track 76.5 -> 161.7 mm, vias 2 -> 0
- net P009: track 104.4 -> 177.8 mm
- net P017: track 136.6 -> 88.0 mm, vias 2 -> 4
- net P022: track 133.8 -> 87.9 mm
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Other:
- board text added: "n36tsu v1.0.0"
- board text removed: "n36tsu v0.1.0"

Commit message: Update PCB wiring (DRC)
Routing:
- net VCC: track 47.3 -> 83.7 mm, vias 0 -> 2
- net GND: track 230.7 -> 263.5 mm, vias 0 -> 2
- net P111: track 251.3 -> 259.4 mm
- net P113: track 222.7 -> 228.0 mm
- net P115: track 268.6 -> 271.2 mm
- net P010: track 212.8 -> 213.5 mm
- net P009: track 177.8 -> 177.1 mm
- net P022: track 87.9 -> 87.4 mm
Other:
- board text added: "n36tsu v1.0.1"
- board text removed: "n36tsu v1.0.0"

Commit message: Modify PCB
Routing:
- net P115: track 271.2 -> 270.4 mm
Changed lines of the file:
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@@
 			(outputformat 1)
 			(mirror no)
-			(drillshape 1)
+			(drillshape 0)
 			(scaleselection 1)
-			(outputdirectory "")
+			(outputdirectory "gerber")
 		)
 	)
@@
 		)
 		(fp_text user "VCC"
-			(at 0.15 18.5 180)
+			(at 0.0645 21.5 0)
 			(unlocked yes)
 			(layer "F.SilkS")
@@
 		)
 		(fp_text user "P017"
-			(at -5.08 18.5 180)
+			(at -5.08 22.5 0)
 			(unlocked yes)
 			(layer "F.SilkS")
@@
 		)
 		(fp_text user "GND"
-			(at 2.62 18.5 180)
+			(at 2.5345 21.5 0)
 			(unlocked yes)
 			(layer "F.SilkS")
@@
 		)
 		(fp_text user "P020"
-			(at -2.48 18.5 180)
+			(at -2.48 22.5 0)
 			(unlocked yes)
 			(layer "F.SilkS")
@@
 		)
 		(fp_text user "P022"
-			(at 5.12 18.5 180)
+			(at 5.12 22.5 0)
 			(unlocked yes)
 			(layer "F.SilkS")
@@
 	)
 	(segment
-		(start 233.5 62.5)
-		(end 205.976771 62.5)
-		(width 0.2)
-		(layer "B.Cu")
-		(net 44)
-	)
-	(segment
-		(start 234.5 61.5)
-		(end 233.5 62.5)
-		(width 0.2)
-		(layer "B.Cu")
-		(net 44)
-	)
-	(segment
 		(start 292 70.5)
 		(end 283 61.5)
@@
 	)
 	(segment
-		(start 293 70.5)
-		(end 292 70.5)
+		(start 204.976771 61.5)
+		(end 199.503853 56.027082)
 		(width 0.2)
 		(layer "B.Cu")
@@
 	)
 	(segment
-		(start 205.976771 62.5)
-		(end 199.503853 56.027082)
+		(start 283 61.5)
+		(end 204.976771 61.5)
 		(width 0.2)
 		(layer "B.Cu")
@@
 	)
 	(segment
-		(start 283 61.5)
-		(end 234.5 61.5)
+		(start 293 70.5)
+		(end 292 70.5)
 		(width 0.2)
 		(layer "B.Cu")
@@
 	)
 	(segment
-		(start 126.6 72)
-		(end 126.1 72.5)
-		(width 0.2)
-		(layer "B.Cu")
-		(net 45)
-	)
-	(segment
-		(start 96.094127 72.5)
-		(end 95.594127 72)
+		(start 122.999316 72)
+		(end 71.6 72)
 		(width 0.2)
 		(layer "B.Cu")
@@
 	)
 	(segment
-		(start 95.594127 72)
-		(end 71.6 72)
+		(start 126.6 72)
+		(end 126.023709 72)
 		(width 0.2)
 		(layer "B.Cu")
@@
 	)
 	(segment
-		(start 126.1 72.5)
-		(end 96.094127 72.5)
+		(start 126.023709 72)
+		(end 125.886776 72.136933)
+		(width 0.2)
+		(layer "B.Cu")
+		(net 45)
+	)
+	(segment
+		(start 125.886776 72.136933)
+		(end 123.136249 72.136933)
+		(width 0.2)
+		(layer "B.Cu")
+		(net 45)
+	)
+	(segment
+		(start 123.136249 72.136933)
+		(end 122.999316 72)
 		(width 0.2)
 		(layer "B.Cu")
@@
 	)
 	(segment
+		(start 204.2455 72.3)
+		(end 201.85 69.9045)
+		(width 0.2)
+		(layer "F.Cu")
+		(net 55)
+	)
+	(segment
 		(start 224.604461 109.004091)
 		(end 224.108552 109.5)
@@
 	)
 	(segment
-		(start 215.5 102.4)
-		(end 215.5 73.131372)
-		(width 0.2)
-		(layer "F.Cu")
-		(net 55)
-	)
-	(segment
 		(start 215.5 73.131372)
 		(end 214.668628 72.3)
@@
 	)
 	(segment
-		(start 204.2455 72.3)
-		(end 201.85 69.9045)
+		(start 215.5 102.4)
+		(end 215.5 73.131372)
 		(width 0.2)
 		(layer "F.Cu")
